File: lib/Kicad/LogUnit.kicad_pcb (KiCad board)
At the start: 2 copper layers, 8 parts, among them U1 ProS3, U3 RFID-RC522

Commit message: PCB done
Parts:
- D1, D2, D3: footprint LED_SMD:LED_0201_0603Metric_Pad0.64x0.40mm_HandSolder -> LED_SMD:LED_0603_1608Metric_Pad1.05x0.95mm_HandSolder
- moved R3 42.7 mm to (107.2, 122.2), turned to -90 degrees
- moved D3 42.0 mm to (107.2, 126.5), turned to 90 degrees
- moved R2 41.0 mm to (111.0, 122.2), turned to -90 degrees
- moved D2 40.2 mm to (111.0, 126.6), turned to 90 degrees
- moved R1 39.8 mm to (114.8, 122.2), turned to -90 degrees
- moved D1 38.6 mm to (114.8, 126.5), turned to 90 degrees
- moved U3 12.6 mm to (114.2, 69.8), turned to -90 degrees
Connections:
- R1 pad 1: Net-(U1-IO1) -> Net-(U1-IO15)
- R2 pad 1: Net-(U1-IO2) -> Net-(U1-IO14)
- R3 pad 1: Net-(U1-IO3) -> Net-(U1-IO13)
- U1 pad 14: unconnected-(U1-IO15-Pad14) -> Net-(U1-IO15)
- U1 pad 15: unconnected-(U1-IO14-Pad15) -> Net-(U1-IO14)
- U1 pad 16: unconnected-(U1-IO13-Pad16) -> Net-(U1-IO13)
- U1 pad 5: Net-(U1-IO1) -> unconnected-(U1-IO1-Pad5)
- U1 pad 6: Net-(U1-IO2) -> unconnected-(U1-IO2-Pad6)
- U1 pad 7: Net-(U1-IO3) -> unconnected-(U1-IO3-Pad7)
Routing:
- net RST: track 0.00 -> 25.4 mm
- net SDA: track 0.00 -> 24.5 mm
- net SCK: track 0.00 -> 16.9 mm
- net Net-(U1-IO15): track 0.00 -> 15.8 mm
- net MISO: track 0.00 -> 15.4 mm
- net Net-(U1-IO14): track 0.00 -> 11.1 mm
- net MOSI: track 0.00 -> 11.0 mm
- net Net-(U1-IO13): track 0.00 -> 6.64 mm
- net GND: track 0.00 -> 4.27 mm, vias 0 -> 2
- net Net-(D2-A): track 0.00 -> 3.34 mm
- net Net-(D3-A): track 0.00 -> 3.25 mm
- net Net-(D1-A): track 0.00 -> 3.25 mm
- added copper zone on F.Cu, net GND

Commit message: updated kicad
Connections:
- U1 pad 25: unconnected-(U1-GND-Pad25) -> GND
- U1 pad 4: unconnected-(U1-3V3-Pad4) -> +3.3V
Routing:
- net +3.3V: track 0.00 -> 20.5 mm
- net GND: track 4.27 -> 8.24 mm, vias 2 -> 4
Changed lines of the file:
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@@
 	(net 27 "MOSI")
 	(net 28 "unconnected-(U1-TX-Pad24)")
-	(net 29 "unconnected-(U1-3V3-Pad4)")
-	(net 30 "unconnected-(U1-LDO2_OUT-Pad12)")
-	(net 31 "unconnected-(U1-IO16-Pad13)")
-	(net 32 "SDA")
-	(net 33 "unconnected-(U1-RST-Pad26)")
-	(net 34 "unconnected-(U1-GND-Pad25)")
-	(net 35 "unconnected-(U1-IO40-Pad20)")
-	(net 36 "MISO")
-	(net 37 "unconnected-(U1-IO38-Pad22)")
-	(net 38 "SCK")
-	(net 39 "unconnected-(U3-IRQ-Pad5)")
-	(net 40 "+3.3V")
+	(net 29 "unconnected-(U1-LDO2_OUT-Pad12)")
+	(net 30 "unconnected-(U1-IO16-Pad13)")
+	(net 31 "SDA")
+	(net 32 "unconnected-(U1-RST-Pad26)")
+	(net 33 "unconnected-(U1-IO40-Pad20)")
+	(net 34 "MISO")
+	(net 35 "unconnected-(U1-IO38-Pad22)")
+	(net 36 "SCK")
+	(net 37 "unconnected-(U3-IRQ-Pad5)")
+	(net 38 "+3.3V")
 	(footprint "Resistor_SMD:R_0402_1005Metric_Pad0.72x0.64mm_HandSolder"
 		(layer "F.Cu")
@@
 			)
 		)
+		(sheetname "Roden")
+		(sheetfile "LogUnit.kicad_sch")
 		(attr through_hole)
 		(fp_rect
@@
 			(layers "*.Cu" "*.Mask")
 			(remove_unused_layers no)
-			(net 29 "unconnected-(U1-3V3-Pad4)")
+			(net 38 "+3.3V")
 			(pinfunction "3V3")
-			(pintype "power_in+no_connect")
+			(pintype "power_in")
 		)
 		(pad "5" thru_hole oval
@@
 			(layers "*.Cu" "*.Mask")
 			(remove_unused_layers no)
-			(net 30 "unconnected-(U1-LDO2_OUT-Pad12)")
+			(net 29 "unconnected-(U1-LDO2_OUT-Pad12)")
 			(pinfunction "LDO2_OUT")
 			(pintype "power_out+no_connect")
@@
 			(layers "*.Cu" "*.Mask")
 			(remove_unused_layers no)
-			(net 31 "unconnected-(U1-IO16-Pad13)")
+			(net 30 "unconnected-(U1-IO16-Pad13)")
 			(pinfunction "IO16")
 			(pintype "bidirectional+no_connect")
@@
 			(layers "*.Cu" "*.Mask")
 			(remove_unused_layers no)
-			(net 35 "unconnected-(U1-IO40-Pad20)")
+			(net 33 "unconnected-(U1-IO40-Pad20)")
 			(pinfunction "IO40")
 			(pintype "bidirectional+no_connect")
@@
 			(layers "*.Cu" "*.Mask")
 			(remove_unused_layers no)
-			(net 37 "unconnected-(U1-IO38-Pad22)")
+			(net 35 "unconnected-(U1-IO38-Pad22)")
 			(pinfunction "IO38")
 			(pintype "bidirectional+no_connect")
@@
 			(layers "*.Cu" "*.Mask")
 			(remove_unused_layers no)
-			(net 34 "unconnected-(U1-GND-Pad25)")
+			(net 1 "GND")
 			(pinfunction "GND")
-			(pintype "power_in+no_connect")
+			(pintype "power_in")
 		)
 		(pad "26" thru_hole oval
@@
 			(layers "*.Cu" "*.Mask")
 			(remove_unused_layers no)
-			(net 33 "unconnected-(U1-RST-Pad26)")
+			(net 32 "unconnected-(U1-RST-Pad26)")
 			(pinfunction "RST")
 			(pintype "input+no_connect")
@@
 			(layers "*.Cu" "*.Mask")
 			(remove_unused_layers no)
-			(net 32 "SDA")
+			(net 31 "SDA")
 			(pinfunction "IO8")
 			(pintype "bidirectional")
@@
 			(layers "*.Cu" "*.Mask")
 			(remove_unused_layers no)
-			(net 38 "SCK")
+			(net 36 "SCK")
 			(pinfunction "IO36")
 			(pintype "bidirectional")
@@
 			(layers "*.Cu" "*.Mask")
 			(remove_unused_layers no)
-			(net 36 "MISO")
+			(net 34 "MISO")
 			(pinfunction "IO37")
 			(pintype "bidirectional")
@@
 			(layers "*.Cu" "*.Mask")
 			(remove_unused_layers no)
-			(net 32 "SDA")
+			(net 31 "SDA")
 			(pinfunction "SS")
 			(pintype "input")
@@
 			(layers "*.Cu" "*.Mask")
 			(remove_unused_layers no)
-			(net 38 "SCK")
+			(net 36 "SCK")
 			(pinfunction "SCK")
 			(pintype "input")
@@
 			(layers "*.Cu" "*.Mask")
 			(remove_unused_layers no)
-			(net 36 "MISO")
+			(net 34 "MISO")
 			(pinfunction "MISO")
 			(pintype "output")
@@
 			(layers "*.Cu" "*.Mask")
 			(remove_unused_layers no)
-			(net 39 "unconnected-(U3-IRQ-Pad5)")
+			(net 37 "unconnected-(U3-IRQ-Pad5)")
 			(pinfunction "IRQ")
 			(pintype "output+no_connect")
@@
 			(layers "*.Cu" "*.Mask")
 			(remove_unused_layers no)
-			(net 40 "+3.3V")
+			(net 38 "+3.3V")
 			(pinfunction "VCC")
 			(pintype "power_in")
@@
 		(drill 0.3)
 		(layers "F.Cu" "B.Cu")
+		(net 1)
+	)
+	(via
+		(at 107.5 79.75)
+		(size 0.6)
+		(drill 0.3)
+		(layers "F.Cu" "B.Cu")
+		(free yes)
+		(net 1)
+	)
+	(via
+		(at 109.25 76.5)
+		(size 0.6)
+		(drill 0.3)
+		(layers "F.Cu" "B.Cu")
+		(free yes)
 		(net 1)
 	)
@@
 	)
 	(segment
+		(start 107.5 78.25)
+		(end 109.25 76.5)
+		(width 0.5)
+		(layer "B.Cu")
+		(net 1)
+	)
+	(segment
+		(start 107.5 79.75)
+		(end 107.5 78.25)
+		(width 0.5)
+		(layer "B.Cu")
+		(net 1)
+	)
+	(segment
 		(start 115.25 82.75)
 		(end 114 84)
@@
 	(segment
 		(start 119.32 89.45)
-		(end 111.75 81.88)
+		(end 105.345 75.475)
 		(width 0.5)
 		(layer "F.Cu")
@@
 	)
 	(segment
-		(start 111.75 81.88)
-		(end 111.75 80.25)
-		(width 0.5)
-		(layer "F.Cu")
-		(net 9)
-	)
-	(segment
-		(start 111.75 80.25)
-		(end 105.345 73.845)
-		(width 0.5)
-		(layer "F.Cu")
-		(net 9)
-	)
-	(segment
-		(start 105.345 73.845)
+		(start 105.345 75.475)
 		(end 105.345 69.83)
 		(width 0.5)
@@
 		(width 0.5)
 		(layer "F.Cu")
-		(net 32)
+		(net 31)
 	)
 	(segment
@@
 		(width 0.5)
 		(layer "F.Cu")
-		(net 32)
+		(net 31)
 	)
 	(segment
@@
 		(width 0.5)
 		(layer "F.Cu")
-		(net 32)
+		(net 31)
 	)
 	(segment
@@
 		(width 0.5)
 		(layer "F.Cu")
-		(net 36)
+		(net 34)
 	)
 	(segment
@@
 		(width 0.5)
 		(layer "F.Cu")
-		(net 36)
+		(net 34)
 	)
 	(segment
@@
 		(width 0.5)
 		(layer "F.Cu")
-		(net 36)
+		(net 34)
 	)
 	(segment
@@
 		(width 0.5)
 		(layer "F.Cu")
-		(net 36)
+		(net 34)
 	)
 	(segment
@@
 		(width 0.5)
 		(layer "B.Cu")
-		(net 36)
+		(net 34)
 	)
 	(segment
@@
 		(width 0.5)
 		(layer "F.Cu")
-		(net 38)
+		(net 36)
 	)
 	(segment
@@
 		(width 0.5)
 		(layer "F.Cu")
-		(net 38)
+		(net 36)
 	)
 	(segment
@@
 		(width 0.5)
 		(layer "F.Cu")
+		(net 36)
+	)
+	(segment
+		(start 102.805 69.83)
+		(end 101 71.635)
+		(width 0.5)
+		(layer "F.Cu")
+		(net 38)
+	)
+	(segment
+		(start 101 86.25)
+		(end 101.66 86.91)
+		(width 0.5)
+		(layer "F.Cu")
+		(net 38)
+	)
+	(segment
+		(start 101.66 86.91)
+		(end 104.08 86.91)
+		(width 0.5)
+		(layer "F.Cu")
+		(net 38)
+	)
+	(segment
+		(start 101 71.635)
+		(end 101 86.25)
+		(width 0.5)
+		(layer "F.Cu")

Commit message: dockerfile 5.0
Parts:
- added C1: C, Capacitor_Tantalum_SMD:CP_EIA-1608-08_AVX-J_Pad1.25x1.05mm_HandSolder, F.Cu at (104.0, 68.0)
- moved U3 0.92 mm to (114.3, 70.8)
Routing:
- net +3.3V: track 20.5 -> 22.5 mm
- net MOSI: track 11.0 -> 10.1 mm
- net SCK: track 16.9 -> 15.9 mm
- net RST: track 25.4 -> 24.5 mm
- net MISO: track 15.4 -> 14.4 mm
- net SDA: track 24.5 -> 23.5 mm
