File: lib/Kicad/LogUnit.kicad_sch (KiCad schematic)
At the start: 8 parts, among them U1 ProS3, U3 RFID-RC522

Commit message: PCB done
Parts:
- D1, D2, D3: footprint LED_SMD:LED_0201_0603Metric_Pad0.64x0.40mm_HandSolder -> LED_SMD:LED_0603_1608Metric_Pad1.05x0.95mm_HandSolder
Connections:
- net at R3.1: now also U1.16 (IO13); no longer U1.7 (IO3)
- net at R1.1: now also U1.14 (IO15); no longer U1.5 (IO1)
- net at R2.1: now also U1.15 (IO14); no longer U1.6 (IO2)
- no-connect marks 1 -> 26
Other:
- moved on the sheet: D1, D2, D3, R1, R2, R3

Commit message: updated kicad
Connections:
- net +3.3V: now also U1.4 (3V3)
- net GND: now also U1.25 (GND)
- no-connect marks 26 -> 24
Other:
- note added: "ESP32-PROS3"
- note added: "LED Lamper"
- note added: "RFID-RC522"
- moved on the sheet: D1, D2, D3, R1, R2, R3

Commit message: dockerfile 5.0
Parts:
- added C1: C, Capacitor_Tantalum_SMD:CP_EIA-1608-08_AVX-J_Pad1.25x1.05mm_HandSolder, symbol Device:C
Connections:
- net +3.3V: now also C1.2
- net GND: now also C1.1
Changed lines of the file:
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@@
 	(paper "A4")
+	(junction
+		(at 106.68 102.87)
+		(diameter 0)
+		(color 0 0 0 0)
+	)
 	(junction
 		(at 154.94 111.76)
@@
 	)
 	(junction
+		(at 106.68 95.25)
+		(diameter 0)
+		(color 0 0 0 0)
+	)
+	(junction
 		(at 185.42 116.84)
 		(diameter 0)
@@
 	(wire
 		(pts
-			(xy 106.68 100.33) (xy 106.68 77.47)
-		)
-		(stroke
-			(width 0)
-			(type default)
-		)
-	)
-	(wire
-		(pts
 			(xy 154.94 111.76) (xy 161.29 111.76)
 		)
@@
 	(wire
 		(pts
+			(xy 109.22 95.25) (xy 109.22 105.41)
+		)
+		(stroke
+			(width 0)
+			(type default)
+		)
+	)
+	(wire
+		(pts
+			(xy 110.49 81.28) (xy 106.68 81.28)
+		)
+		(stroke
+			(width 0)
+			(type default)
+		)
+	)
+	(wire
+		(pts
+			(xy 106.68 81.28) (xy 106.68 77.47)
+		)
+		(stroke
+			(width 0)
+			(type default)
+		)
+	)
+	(wire
+		(pts
+			(xy 106.68 95.25) (xy 109.22 95.25)
+		)
+		(stroke
+			(width 0)
+			(type default)
+		)
+	)
+	(wire
+		(pts
 			(xy 181.61 116.84) (xy 185.42 116.84)
 		)
@@
 	(wire
 		(pts
+			(xy 97.79 95.25) (xy 106.68 95.25)
+		)
+		(stroke
+			(width 0)
+			(type default)
+		)
+	)
+	(wire
+		(pts
+			(xy 110.49 102.87) (xy 110.49 81.28)
+		)
+		(stroke
+			(width 0)
+			(type default)
+		)
+	)
+	(wire
+		(pts
 			(xy 185.42 109.22) (xy 185.42 116.84)
 		)
@@
 	(wire
 		(pts
+			(xy 97.79 100.33) (xy 100.33 100.33)
+		)
+		(stroke
+			(width 0)
+			(type default)
+		)
+	)
+	(wire
+		(pts
 			(xy 153.67 106.68) (xy 154.94 106.68)
 		)
@@
 	(wire
 		(pts
+			(xy 106.68 102.87) (xy 110.49 102.87)
+		)
+		(stroke
+			(width 0)
+			(type default)
+		)
+	)
+	(wire
+		(pts
 			(xy 161.29 101.6) (xy 161.29 106.68)
 		)
@@
 	(wire
 		(pts
-			(xy 97.79 100.33) (xy 106.68 100.33)
+			(xy 100.33 102.87) (xy 106.68 102.87)
 		)
 		(stroke
@@
 	(wire
 		(pts
+			(xy 100.33 100.33) (xy 100.33 102.87)
+		)
+		(stroke
+			(width 0)
+			(type default)
+		)
+	)
+	(wire
+		(pts
 			(xy 185.42 101.6) (xy 185.42 109.22)
 		)
@@
 	(wire
 		(pts
-			(xy 97.79 95.25) (xy 109.22 95.25)
-		)
-		(stroke
-			(width 0)
-			(type default)
-		)
-	)
-	(wire
-		(pts
 			(xy 154.94 106.68) (xy 161.29 106.68)
 		)
@@
 		(pts
 			(xy 158.75 81.28) (xy 158.75 77.47)
-		)
-		(stroke
-			(width 0)
-			(type default)
-		)
-	)
-	(wire
-		(pts
-			(xy 109.22 95.25) (xy 109.22 105.41)
 		)
 		(stroke
@@
 					(unit 1)
 				)
+			)
+		)
+	)
+	(symbol
+		(lib_id "Device:C")
+		(at 106.68 99.06 0)
+		(unit 1)
+		(exclude_from_sim no)
+		(in_bom yes)
+		(on_board yes)
+		(dnp no)
+		(property "Reference" "C1"
+			(at 104.14 96.52 0)
+			(effects
+				(font
+					(size 1.27 1.27)
+				)
+				(justify left)
+				(hide yes)
+			)
+		)
+		(property "Value" "C"
+			(at 104.14 96.52 0)
+			(effects
+				(font
+					(size 1.27 1.27)
+				)
+				(justify left)
+			)
+		)
+		(property "Footprint" "Capacitor_Tantalum_SMD:CP_EIA-1608-08_AVX-J_Pad1.25x1.05mm_HandSolder"
+			(at 107.6452 102.87 0)
+			(effects
+				(font
+					(size 1.27 1.27)
+				)
+				(hide yes)
+			)
+		)
+		(property "Datasheet" "~"
+			(at 106.68 99.06 0)
+			(effects
+				(font
+					(size 1.27 1.27)
+				)
+				(hide yes)
+			)
+		)
+		(property "Description" "Unpolarized capacitor"
+			(at 106.68 99.06 0)
+			(effects
+				(font
+					(size 1.27 1.27)
+				)
+				(hide yes)
+			)
+		)
+		(pin "2"
+		)
+		(pin "1"
+		)
+		(instances
+			(project "LogUnit"
+				(path "/9d88098b-233a-4b6f-bb56-5045204966fd"
+					(reference "C1")
+					(unit 1)
+				)
